File: hw/ktwinkler-r2025-11/ktwinkler-r2025-11.kicad_pcb (KiCad board)
At the start: 2 copper layers, 38 x 15 mm, 14 parts

Commit message: pushing ideas around
Parts:
- removed the REF** at (133.1, 75.7)
- removed the REF** at (85.5, 106.3)
- removed the REF** at (154.3, 77.1)
- removed the REF** at (141.8, 65.6)
- removed the REF** at (125.7, 80.1)
- removed the REF** at (133.8, 77.2)
- removed the REF** at (130.8, 82.2)
- removed the REF** at (128.2, 82.5)
- removed the REF** at (144.4, 80.8)
- removed the REF** at (134.4, 81.7)
- removed the REF** at (146.6, 72.8)
- removed the REF** at (125.6, 82.3)
- removed the REF** at (138.2, 72.7)
- removed the REF** at (156.3, 71.6)
- added C1: 100nF, Capacitor_SMD:C_0603_1608Metric, F.Cu at (123.2, 81.3)
- added C2: 100nF, Capacitor_SMD:C_0603_1608Metric, F.Cu at (123.2, 83.9)
- added C3: 100nF, Capacitor_SMD:C_0603_1608Metric, F.Cu at (140.6, 73.3)
- added C4: 100nF, Capacitor_SMD:C_0603_1608Metric, F.Cu at (140.6, 75.8)
- added C5: 100nF, Capacitor_SMD:C_0603_1608Metric, F.Cu at (149.8, 74.0)
- added J1: USB_C_Receptacle_USB2.0_16P, Connector_USB:USB_C_Receptacle_GCT_USB4110, F.Cu at (143.1, 82.5)
- added J2: Conn_01x03, Connector_PinHeader_2.54mm:PinHeader_1x03_P2.54mm_Vertical, F.Cu at (154.7, 71.8)
- added J3: Conn_01x03, TerminalBlock_Phoenix:TerminalBlock_Phoenix_MPT-0,5-3-2.54_1x03_P2.54mm_Horizontal, F.Cu at (154.6, 76.8)
- added J4: Conn_01x01, Connector_Wire:SolderWire-0.5sqmm_1x01_D0.9mm_OD2.1mm, F.Cu at (126.2, 83.3)
- added J5: Conn_01x01, Connector_Wire:SolderWire-0.5sqmm_1x01_D0.9mm_OD2.1mm, F.Cu at (155.8, 82.8)
- added L1: 1uH, Inductor_SMD:L_1206_3216Metric, F.Cu at (129.3, 82.7)
- added R1: 5k1, Resistor_SMD:R_0603_1608Metric, F.Cu at (151.9, 81.1)
- added R2: 5k1, Resistor_SMD:R_0603_1608Metric, F.Cu at (152.1, 83.5)
- added R3: 0R, Resistor_SMD:R_0603_1608Metric, F.Cu at (122.2, 72.7)
- added REF**: Val**, wch-antenna:ANT-F-3-2.4G-1.6MM-FR4-WCH, F.Cu at (121.8, 75.3)
- added SW5: MODE, Button_Switch_SMD:SW_SPST_TL3342, F.Cu at (135.4, 77.5)
- added U1: TPS631000DRLR, Package_TO_SOT_SMD:SOT-583-8, F.Cu at (133.0, 83.0)
- added U2: LK116, Package_TO_SOT_SMD:SOT-23-6, F.Cu at (146.0, 73.0)
- added U3: ESP32-C3FH4, Package_DFN_QFN:QFN-32-1EP_5x5mm_P0.5mm_EP3.7x3.7mm, F.Cu at (126.8, 75.7)
- added Y1: 40M, Crystal:Crystal_SMD_2016-4Pin_2.0x1.6mm, F.Cu at (135.0, 73.4)
- added Y2: X1A0001210005, Crystal:Crystal_SMD_MicroCrystal_CM9V-T1A-2Pin_1.6x1.0mm, F.Cu at (132.1, 71.5)
Other:
- board text added: "PLENTTTTTTTY OF ROOOOM"
- board text added: "Will USB fit? or will it be pins for uart?"
- board text added: "thefuckin button goes where?!"
