File: hw/ktwinkler-r2025-11/ktwinkler-r2025-11.kicad_sch (KiCad schematic)
At the start: 0 parts

Commit message: pushing ideas around
Parts:
- added AE1: Antenna_Dipole, symbol Device:Antenna_Dipole
- added C1, C2, C3, C4, C5: 100nF, Capacitor_SMD:C_0603_1608Metric, symbol karl-atomic-basic:KC0603_100nF
- added J1: USB_C_Receptacle_USB2.0_16P, Connector_USB:USB_C_Receptacle_GCT_USB4110, symbol Connector:USB_C_Receptacle_USB2.0_16P
- added J2: Conn_01x03, Connector_PinHeader_2.54mm:PinHeader_1x03_P2.54mm_Vertical, symbol Connector_Generic:Conn_01x03
- added J3: Conn_01x03, TerminalBlock_Phoenix_MPT-0,5-3-2.54_1x03_P2.54mm_Horizontal, symbol Connector_Generic:Conn_01x03
- added J4, J5: Conn_01x01, Connector_Wire:SolderWire-0.5sqmm_1x01_D0.9mm_OD2.1mm, symbol Connector_Generic:Conn_01x01
- added L1: 1uH, Inductor_SMD:L_1206_3216Metric, symbol Device:L_Small
- added R1, R2: 5k1, Resistor_SMD:R_0603_1608Metric, symbol karl-atomic-basic:KR0603_5k1
- added R3: 0R, Resistor_SMD:R_0603_1608Metric, symbol karl-atomic-basic:KR0603_0R
- added SW5: MODE, Button_Switch_SMD:SW_SPST_TL3342, symbol Switch:SW_Push
- added U1: TPS631000DRLR, Package_TO_SOT_SMD:SOT-583-8, symbol karl-parts:TPS631000DRLR
- added U2: LK116, Package_TO_SOT_SMD:SOT-23-6, symbol karl-parts:LK116
- added U3: ESP32-C3FH4, Package_DFN_QFN:QFN-32-1EP_5x5mm_P0.5mm_EP3.7x3.7mm, symbol karl-parts:ESP32-C3FH4
- added Y1: 40M, Crystal:Crystal_SMD_2016-4Pin_2.0x1.6mm, symbol Device:Crystal_GND24_Small
- added Y2: X1A0001210005, Crystal:Crystal_SMD_MicroCrystal_CM9V-T1A-2Pin_1.6x1.0mm, symbol karl-parts:X1A0001210005
Connections:
- new net: AE1.1, R3.2
- new net: J1.A1 (GND), J1.A12 (GND), J1.B1 (GND), J1.B12 (GND)
- new net: J1.A4 (VBUS), J1.A9 (VBUS), J1.B4 (VBUS), J1.B9 (VBUS)
- new net: R3.1, U3.1 (LNA_IN)
- new net: U3.2 (VDD3P3), U3.3 (VDD3P3)
- new net: U3.31 (VDDA), U3.32 (VDDA)
- new net: L1.1, U1.2 (L2)
- new net: L1.2, U1.3 (L1)
- new net +BATT: J4.1 (Pin_1)
- new net GND: J5.1 (Pin_1)
Other:
- note added: "2/3 cells AA, with shitty 1.2V nimh, flat, we need buck boost from ~2V to ~4.6V Decent parts on JLC, under $0.60, with >1A RT6150A (0.8A, 1MHz) TPS63802DLAR 3A, promises 0.47uH tiny L TPS63020 4A, 2.4MHz (bigger package) TPS631000 (great stock, looks good)"
- note added: "2016 is the cheapest smallest 40M crystal if you do this yourself the hard way Do we _realllllly_ need a 32k? yeahhhh, that's the point right?"
- note added: "ESP32x in 13.2x16.6mm modules: ESP32-C6-MINI-1-N4 - well stocked, $4 (wifi+btle+802.15.4) ESP32-C61-MINI-1 - no stock ESP32-C3-MINI-1-H4X - well stocked, $3 (wifi+btle) ESP8684-MINI-1-H4 - some stock, $2 (wifi+btle) ESP32-H2-MINI-1 - no stock (btle+802.15.4 only) ESP32-PICO-MINI-02-N8R2 - well stocked, $5 (wifi+bt+btle) So... C6 or C3? fuck matter... C3 is fine :) So.. C6 has the low power coproc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"
- note added: "Separate because these are battery contacts in the replacement board"
- note added: "TODO: use 0402 TODO: will a vert mount fit? (prb too tall?)"
- note added: "~4V, peak power is.... what? 0.4 2W? Connect the boards up again?"
- note removed: "2016 is the cheapest smallest 40M crystal if you do this yourself the hard way"
- note removed: "ESP32x in 13.2x16.6mm modules: ESP32-C6-MINI-1-N4 - well stocked, $4 (wifi+btle+802.15.4) ESP32-C61-MINI-1 - no stock ESP32-C3-MINI-1-H4X - well stocked, $3 (wifi+btle) ESP8684-MINI-1-H4 - some stock, $2 (wifi+btle) ESP32-H2-MINI-1 - no stock (btle+802.15.4 only) ESP32-PICO-MINI-02-N8R2 - well stocked, $5 (wifi+bt+btle) So... C6 or C3? fuck matter... C3 is fine :)"

Commit message: make a v2 idea, mroe experiments, less product...
Other:
- note added: "Replaces anti-parallel led driver in battery pack string lights. Adds wifi/btle for control WILL be more expensive Aim to fit in the same casings. Use an esp32 family to make easier for "community" hacking rather than el cheapo chinesium bluetooth gear But you, CH572, or CH592, or CH582 would be _small_ and _lower power_ and _cheaper_? 572d is 40c, 3x3mm, 20pins, more than enough, but fuck all ra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"
- note removed: "Replaces anti-parallel led driver in battery pack string lights. Adds wifi/btle for control WILL be more expensive Aim to fit in the same casings. Use an esp32 family to make easier for "community" hacking rather than el cheapo chinesium bluetooth gear"
Changed lines of the file:
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@@
 	(generator_version "9.0")
 	(paper "A4")
-	(text "Replaces anti-parallel led driver in battery pack string lights.\nAdds wifi/btle for control\nWILL be more expensive\nAim to fit in the same casings.\nUse an esp32 family to make easier for \"community\" hacking rather than\nel cheapo chinesium bluetooth gear"
+	(text "Replaces anti-parallel led driver in battery pack string lights.\nAdds wifi/btle for control\nWILL be more expensive\nAim to fit in the same casings.\nUse an esp32 family to make easier for \"community\" hacking rather than\nel cheapo chinesium bluetooth gear\nBut you, CH572, or CH592, or CH582 would be _small_ and _lower power_ and _cheaper_?\n572d is 40c, 3x3mm, 20pins, more than enough, but fuck all ram.\n582f is 4x4mm, 28pins, we've used it before.\n584f is still only 90c, 4x4, 32pins"
 		(exclude_from_sim no)
 		(at 29.972 46.482 0)
