File: hw/ktwinkler-multi-r2025-12/ktwinkler-multi-r2025-12.kicad_pcb (KiCad board)
At the start: 2 copper layers, 38 x 15 mm, 21 parts, among them J1 USB_C_Receptacle_USB2.0_16P, J2 Conn_01x03, J3 Conn_01x03, J4 Conn_01x01, J5 Conn_01x01, SW5 MODE, U1 TPS631000DRLR, U2 LK116, U3 ESP32-C3FH4, Y1 40M, Y2 X1A0001210005

Commit message: pushing onwards like a madlad
Parts:
- removed J3: Conn_01x03, TerminalBlock_Phoenix:TerminalBlock_Phoenix_MPT-0,5-3-2.54_1x03_P2.54mm_Horizontal
- removed REF**: Val**, wch-antenna:ANT-F-3-2.4G-1.6MM-FR4-WCH
- added AE2: Antenna_Loop, wch-antenna:ANT-F-1-2.4G-1.6MM-FR4-WCH-FLIP, F.Cu at (223.0, 79.1)
- added C10: 22pF, Capacitor_SMD:C_0402_1005Metric, F.Cu at (187.8, 80.0)
- added C11: 22pF, Capacitor_SMD:C_0402_1005Metric, F.Cu at (187.8, 82.0)
- added C12: 22pF, Capacitor_SMD:C_0402_1005Metric, F.Cu at (187.8, 84.0)
- added C13: 100nF, Capacitor_SMD:C_0402_1005Metric, F.Cu at (187.8, 85.9)
- added C14: 100nF, Capacitor_SMD:C_0402_1005Metric, F.Cu at (187.8, 87.9)
- added C15: 22uF, Capacitor_SMD:C_0805_2012Metric, F.Cu at (115.0, 141.2)
- added C16: 22uF, Capacitor_SMD:C_0805_2012Metric, F.Cu at (107.0, 144.5)
- added C17: 1uF, Capacitor_SMD:C_0603_1608Metric, F.Cu at (191.3, 95.5)
- added C18: 2.2pF, Capacitor_SMD:C_0402_1005Metric, F.Cu at (187.8, 89.9)
- added C6: 100nF, Capacitor_SMD:C_0402_1005Metric, F.Cu at (101.0, 125.7)
- added C7: 1uF, Capacitor_SMD:C_0603_1608Metric, F.Cu at (191.3, 90.5)
- added C8: 1uF, Capacitor_SMD:C_0603_1608Metric, F.Cu at (191.3, 93.0)
- added C9: 22pF, Capacitor_SMD:C_0402_1005Metric, F.Cu at (187.8, 78.1)
- added D1: SS34, Diode_SMD:D_SMA, F.Cu at (121.2, 145.2)
- added J10: Conn_01x06, Connector_PinHeader_2.54mm:PinHeader_1x06_P2.54mm_Vertical, F.Cu at (213.5, 77.4)
- added J11: Conn_01x02, Connector_Phoenix_MC:PhoenixContact_MCV_1,5_2-G-3.81_1x02_P3.81mm_Vertical, F.Cu at (138.0, 100.0)
- added J6: Conn_01x02, Connector_Phoenix_MC:PhoenixContact_MCV_1,5_2-G-3.81_1x02_P3.81mm_Vertical, F.Cu at (116.0, 100.0)
- added J7: Conn_01x02, Connector_Phoenix_MC:PhoenixContact_MCV_1,5_2-G-3.81_1x02_P3.81mm_Vertical, F.Cu at (105.0, 100.0)
- added J8: Conn_01x02, Connector_Phoenix_MC:PhoenixContact_MCV_1,5_2-G-3.81_1x02_P3.81mm_Vertical, F.Cu at (127.0, 100.0)
- added J9: BWU.FL-IPEX1, Connector_Coaxial:U.FL_Hirose_U.FL-R-SMT-1_Vertical, F.Cu at (102.0, 116.5)
- added L2: 1nH, Inductor_SMD:L_0402_1005Metric, F.Cu at (200.3, 76.1)
- added R10: 10k, Resistor_SMD:R_0402_1005Metric, F.Cu at (200.3, 86.0)
- added R11: 10k, Resistor_SMD:R_0402_1005Metric, F.Cu at (203.2, 76.1)
- added R12: 10k, Resistor_SMD:R_0402_1005Metric, F.Cu at (203.2, 78.1)
- added R13: 10k, Resistor_SMD:R_0402_1005Metric, F.Cu at (203.2, 80.1)
- added R14: 10k, Resistor_SMD:R_0402_1005Metric, F.Cu at (212.9, 101.8)
- added R15: 0R, Resistor_SMD:R_0402_1005Metric, F.Cu at (203.2, 82.1)
- added R16: 0R, Resistor_SMD:R_0402_1005Metric, F.Cu at (203.2, 84.1)
- added R17: 0R, Resistor_SMD:R_0402_1005Metric, F.Cu at (226.8, 84.1)
- added R18: 0R, Resistor_SMD:R_0402_1005Metric, F.Cu at (226.8, 86.1)
- added R19: 0R, Resistor_SMD:R_0402_1005Metric, F.Cu at (226.8, 88.1)
- added R4: 0R, Resistor_SMD:R_0402_1005Metric, F.Cu at (200.3, 80.1)
- added R5: 0R, Resistor_SMD:R_0402_1005Metric, F.Cu at (200.3, 82.1)
- added R6: 0R, Resistor_SMD:R_0402_1005Metric, F.Cu at (109.5, 144.3)
- added R7: 39k, Resistor_SMD:R_0402_1005Metric, F.Cu at (111.0, 144.0)
- added R8: 220k, Resistor_SMD:R_0402_1005Metric, F.Cu at (111.5, 141.5)
- added R9: 470R, Resistor_SMD:R_0402_1005Metric, F.Cu at (200.3, 84.1)
- added SW1: RESET, Button_Switch_SMD:SW_SPST_TL3342, F.Cu at (194.0, 78.6)
- added SW2: BOOT, Button_Switch_SMD:SW_SPST_TL3342, F.Cu at (194.0, 85.7)
- added SW4: BOOT, Button_Switch_SMD:SW_SPST_TL3342, F.Cu at (220.6, 86.7)
- added SW6: RESET_CH, Button_Switch_SMD:SW_SPST_TL3342, F.Cu at (220.6, 93.7)
- added U4: T1016H, Package_TO_SOT_SMD:SOT-23-6, F.Cu at (107.4, 109.7)
- added U5: AD116, Package_TO_SOT_SMD:SOT-23-6, F.Cu at (128.6, 109.5)
- added U6: FM116C, Package_TO_SOT_SMD:SOT-23-6, F.Cu at (139.4, 109.2)
- added U7: SRV05-4, Package_TO_SOT_SMD:SOT-23-6, F.Cu at (130.4, 141.6)
- added Y3: XL2EL89CPI-111YLC-40M, Crystal:Crystal_SMD_3225-4Pin_3.2x2.5mm, F.Cu at (201.4, 96.6)
- added Y4: Crystal_32M_2016_XTM20032000DT00351005, Crystal:Crystal_SMD_2016-4Pin_2.0x1.6mm, F.Cu at (227.4, 94.3)
- C1: value 100nF -> 22uF; footprint Capacitor_SMD:C_0603_1608Metric -> Capacitor_SMD:C_0805_2012Metric
- C2, C3, C4, C5: footprint Capacitor_SMD:C_0603_1608Metric -> Capacitor_SMD:C_0402_1005Metric
- J2: value Conn_01x03 -> Conn_01x02; footprint Connector_PinHeader_2.54mm:PinHeader_1x03_P2.54mm_Vertical -> Connector_PinHeader_2.54mm:PinHeader_1x02_P2.54mm_Vertical
- J4: value Conn_01x01 -> Conn_01x02; footprint Connector_Wire:SolderWire-0.5sqmm_1x01_D0.9mm_OD2.1mm -> Connector_Phoenix_MC:PhoenixContact_MCV_1,5_2-G-3.81_1x02_P3.81mm_Vertical
- J5: value Conn_01x01 -> Conn_01x03; footprint Connector_Wire:SolderWire-0.5sqmm_1x01_D0.9mm_OD2.1mm -> Connector_PinHeader_2.54mm:PinHeader_1x03_P2.54mm_Vertical
- R1, R2, R3: footprint Resistor_SMD:R_0603_1608Metric -> Resistor_SMD:R_0402_1005Metric
- U2: value LK116 -> FM116C
- Y1: value 40M -> Q13FC13500004; footprint Crystal:Crystal_SMD_2016-4Pin_2.0x1.6mm -> Crystal:Crystal_SMD_3215-2Pin_3.2x1.5mm
- Y2: value X1A0001210005 -> Q13FC13500004; footprint Crystal:Crystal_SMD_MicroCrystal_CM9V-T1A-2Pin_1.6x1.0mm -> Crystal:Crystal_SMD_3215-2Pin_3.2x1.5mm
- moved Y1 94.5 mm to (227.9, 90.8)
- moved J2 86.1 mm to (118.2, 149.8), turned to -90 degrees
- moved Y2 78.4 mm to (206.6, 96.0)
- moved R3 78.2 mm to (200.3, 78.1)
- moved SW5 74.3 mm to (149.2, 150.5)
- moved J4 70.0 mm to (109.7, 151.4), turned to 180 degrees
- moved J1 68.6 mm to (132.2, 150.2)
- moved C2 65.0 mm to (187.8, 76.1)
- moved R1 64.9 mm to (126.3, 140.8)
- moved R2 64.6 mm to (126.3, 142.7)
- moved U1 63.8 mm to (107.6, 141.4), turned to -90 degrees
- moved C1 60.1 mm to (118.0, 141.2), turned to -90 degrees
- moved L1 59.5 mm to (107.1, 137.9), turned to 180 degrees
- moved J5 51.4 mm to (206.9, 77.4)
- moved U3 46.4 mm to (151.5, 115.0)
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Connections:
- net Net-(J1-VBUS-PadA4) renamed /power/VBUS
- C1 pad 1: unconnected-(C1-Pad1) -> +3V3
- C1 pad 2: unconnected-(C1-Pad2) -> GND
- C2 pad 1: unconnected-(C2-Pad1) -> +3V3
- C2 pad 2: unconnected-(C2-Pad2) -> GND
- C3 pad 1: unconnected-(C3-Pad1) -> Net-(J8-Pin_2)
- C3 pad 2: unconnected-(C3-Pad2) -> Net-(J8-Pin_1)
- C4 pad 1: unconnected-(C4-Pad1) -> Net-(J7-Pin_2)
- C4 pad 2: unconnected-(C4-Pad2) -> Net-(J7-Pin_1)
- C5 pad 1: unconnected-(C5-Pad1) -> Net-(J6-Pin_2)
- C5 pad 2: unconnected-(C5-Pad2) -> Net-(J6-Pin_1)
- J1 pad A1: Net-(J1-GND-PadA1) -> GND
- J1 pad A12: Net-(J1-GND-PadA1) -> GND
- J1 pad A5: unconnected-(J1-CC1-PadA5) -> Net-(J1-CC1)
- J1 pad A6: unconnected-(J1-D+-PadA6) -> USBDP
- J1 pad A7: unconnected-(J1-D--PadA7) -> USBDM
- J1 pad B1: Net-(J1-GND-PadA1) -> GND
- J1 pad B12: Net-(J1-GND-PadA1) -> GND
- J1 pad B5: unconnected-(J1-CC2-PadB5) -> Net-(J1-CC2)
- J1 pad B6: unconnected-(J1-D+-PadB6) -> USBDP
- J1 pad B7: unconnected-(J1-D--PadB7) -> USBDM
- J1 pad S1: unconnected-(J1-SHIELD-PadS1) -> GND
- J2 pad 1: unconnected-(J2-Pin_1-Pad1) -> GND
- J2 pad 2: unconnected-(J2-Pin_2-Pad2) -> +BATT
- J4 pad 1: +BATT -> GND
- R1 pad 1: unconnected-(R1-Pad1) -> Net-(J1-CC1)
- R1 pad 2: unconnected-(R1-Pad2) -> GND
- R2 pad 1: unconnected-(R2-Pad1) -> Net-(J1-CC2)
- R2 pad 2: unconnected-(R2-Pad2) -> GND
- R3 pad 1: Net-(U3-LNA_IN) -> Net-(C18-Pad1)
- SW5 pad 1: unconnected-(SW5-Pad1) -> GND
- SW5 pad 2: unconnected-(SW5-Pad2) -> /MODE
- U1 pad 1: unconnected-(U1-VOUT-Pad1) -> +3V3
- U1 pad 4: unconnected-(U1-VIN-Pad4) -> +BATT
- U1 pad 5: unconnected-(U1-EN-Pad5) -> +BATT
- U1 pad 6: unconnected-(U1-MODE-Pad6) -> Net-(U1-MODE)
- U1 pad 7: unconnected-(U1-GND-Pad7) -> GND
- U1 pad 8: unconnected-(U1-FB-Pad8) -> Net-(U1-FB)
- U2 pad 1: unconnected-(U2-OUTB-Pad1) -> Net-(J6-Pin_1)
- U2 pad 2: unconnected-(U2-GND-Pad2) -> GND
- U2 pad 3: unconnected-(U2-INB-Pad3) -> /ch584/PWM4
- U2 pad 4: unconnected-(U2-INA-Pad4) -> /ch584/PWM3
- U2 pad 5: unconnected-(U2-VDD-Pad5) -> +BATT
- U2 pad 6: unconnected-(U2-OUTA-Pad6) -> Net-(J6-Pin_2)
- U3 pad 10: unconnected-(U3-MTDI-Pad10) -> /esp32/PWM8
- U3 pad 11: unconnected-(U3-VDD3P3_RTC-Pad11) -> +3V3
- U3 pad 14: unconnected-(U3-GPIO8-Pad14) -> Net-(U3-GPIO8)
- U3 pad 15: unconnected-(U3-GPIO9-Pad15) -> Net-(U3-GPIO9)
- U3 pad 16: unconnected-(U3-GPIO10-Pad16) -> /esp32/PWM7
- U3 pad 17: unconnected-(U3-VDD3P3_CPU-Pad17) -> +3V3
- U3 pad 18: unconnected-(U3-VDD_SPI-Pad18) -> +3V3
- U3 pad 19: unconnected-(U3-SPIHD-Pad19) -> /ch584/PWM1
- U3 pad 2: Net-(U3-VDD3P3-Pad2) -> +3V3
- U3 pad 20: unconnected-(U3-SPIWP-Pad20) -> /ch584/PWM2
- U3 pad 21: unconnected-(U3-SPICS0-Pad21) -> /ch584/PWM3
- U3 pad 22: unconnected-(U3-SPICLK-Pad22) -> /ch584/PWM4
- U3 pad 23: unconnected-(U3-SPID-Pad23) -> /ch584/PWM5
- U3 pad 24: unconnected-(U3-SPIQ-Pad24) -> /ch584/PWM6
- U3 pad 25: unconnected-(U3-GPIO18-Pad25) -> Net-(U3-GPIO18)
- U3 pad 26: unconnected-(U3-GPIO19-Pad26) -> Net-(U3-GPIO19)
- U3 pad 27: unconnected-(U3-U0RXD-Pad27) -> Net-(J5-Pin_2)
- U3 pad 28: unconnected-(U3-U0TXD-Pad28) -> Net-(U3-U0TXD)
- U3 pad 29: unconnected-(U3-XTAL_N-Pad29) -> Net-(U3-XTAL_N)
- U3 pad 3: Net-(U3-VDD3P3-Pad2) -> +3V3
- U3 pad 30: unconnected-(U3-XTAL_P-Pad30) -> Net-(U3-XTAL_P)
- U3 pad 31: Net-(U3-VDDA-Pad31) -> +3V3
- U3 pad 32: Net-(U3-VDDA-Pad31) -> +3V3
- U3 pad 33: unconnected-(U3-GND-Pad33) -> GND
- U3 pad 4: unconnected-(U3-XTAL_32K_P-Pad4) -> Net-(U3-XTAL_32K_P)
- U3 pad 5: unconnected-(U3-XTAL_32K_N-Pad5) -> Net-(U3-XTAL_32K_N)
- U3 pad 6: unconnected-(U3-GPIO2-Pad6) -> Net-(U3-GPIO2)
- U3 pad 7: unconnected-(U3-CHIP_EN-Pad7) -> Net-(U3-CHIP_EN)
- U3 pad 8: unconnected-(U3-GPIO3-Pad8) -> /MODE
- Y1 pad 1: unconnected-(Y1-Pad1) -> Net-(U8B-PA11_X32KO_TMR2)
- Y1 pad 2: unconnected-(Y1-Pad2) -> Net-(U8B-PA10_X32KI_TMR1)
- Y2 pad 1: unconnected-(Y2-Pad1) -> Net-(U3-XTAL_32K_N)
- Y2 pad 2: unconnected-(Y2-Pad2) -> Net-(U3-XTAL_32K_P)
Other:
- board outline removed
- board text removed: "thefuckin button goes where?!"

Commit message: ready for scope creep
I think the schematic is ... mostly ok?  I need to decide how much of
the han p1 port scope creep to bother doing, or not...

I've roughyl blocked out the board, seems as good as any?
Parts:
- removed R13: 10k, Resistor_SMD:R_0402_1005Metric
- removed R17, R18: 0R, Resistor_SMD:R_0402_1005Metric
- removed SW4: BOOT, Button_Switch_SMD:SW_SPST_TL3342
- removed SW6: RESET_CH, Button_Switch_SMD:SW_SPST_TL3342
- removed U7: SRV05-4, Package_TO_SOT_SMD:SOT-23-6
- removed Y3: XL2EL89CPI-111YLC-40M, Crystal:Crystal_SMD_3225-4Pin_3.2x2.5mm
- added AE1: Antenna_lolpole, RF_Experiments:ANT-YOLOPOLE, F.Cu at (100.0, 125.0)
- added C19: 1uF, Capacitor_SMD:C_0603_1608Metric, F.Cu at (146.8, 120.5)
- added C20: 100nF, Capacitor_SMD:C_0402_1005Metric, F.Cu at (141.0, 125.2)
- added C22: 1uF, Capacitor_SMD:C_0603_1608Metric, F.Cu at (149.8, 124.5)
- added J12: Connector_HAN_P1, Connector_RJ:RJ25_Wayconn_MJEA-660X1_Horizontal, F.Cu at (148.1, 100.3)
- added J13: Conn_01x02, TestPoint:TestPoint_2Pads_Pitch2.54mm_Drill0.8mm, F.Cu at (137.8, 103.5)
- added J14: Conn_01x02, TestPoint:TestPoint_2Pads_Pitch2.54mm_Drill0.8mm, F.Cu at (116.0, 103.8)
- added J15: Conn_01x02, TestPoint:TestPoint_2Pads_Pitch2.54mm_Drill0.8mm, F.Cu at (105.0, 104.0)
- added J16: Conn_01x02, TestPoint:TestPoint_2Pads_Pitch2.54mm_Drill0.8mm, F.Cu at (126.8, 104.0)
- added J3: Conn_01x04, Connector_PinHeader_2.54mm:PinHeader_1x04_P2.54mm_Vertical, F.Cu at (146.4, 131.4)
- added JP1: KJumper_3, Connector_PinHeader_2.54mm:PinHeader_1x03_P2.54mm_Vertical, F.Cu at (128.2, 125.9)
- added JP2: KJumper_3, Connector_PinHeader_2.54mm:PinHeader_1x03_P2.54mm_Vertical, F.Cu at (132.8, 125.9)
- added JP3: LocalPower, TestPoint:TestPoint_2Pads_Pitch2.54mm_Drill0.8mm, F.Cu at (137.5, 112.0)
- added R20: 10k, Resistor_SMD:R_0402_1005Metric, F.Cu at (148.2, 140.0)
- added U8: CH584F, Package_DFN_QFN:QFN-32-1EP_4x4mm_P0.4mm_EP2.65x2.65mm, F.Cu at (145.2, 125.5)
- added U9: GM8023B, Package_TO_SOT_SMD:SOT-23-6, F.Cu at (132.3, 110.8)
- added Y5: 32M, Crystal:Crystal_SMD_2016-4Pin_2.0x1.6mm, F.Cu at (151.1, 128.9)
- J1: footprint Connector_USB:USB_C_Receptacle_GCT_USB4110 -> Connector_USB:USB_C_Receptacle_GCT_USB4105-xx-A_16P_TopMnt_Horizontal
- J11, J4, J6, J7, J8: footprint Connector_Phoenix_MC:PhoenixContact_MCV_1,5_2-G-3.81_1x02_P3.81mm_Vertical -> Connector_Phoenix_MC:PhoenixContact_MC_1,5_2-G-3.5_1x02_P3.50mm_Horizontal
- R4, R5: value 0R -> 22R
- R6: value 0R -> 10k
- U6: value FM116C -> Protection_H5VU25UC; footprint Package_TO_SOT_SMD:SOT-23-6 -> Package_DFN_QFN:Diodes_UDFN-10_1.0x2.5mm_P0.5mm
- Y1: value Q13FC13500004 -> 40M; footprint Crystal:Crystal_SMD_3215-2Pin_3.2x1.5mm -> Crystal:Crystal_SMD_2016-4Pin_2.0x1.6mm
- Y2: value Q13FC13500004 -> 32k
- Y4: value Crystal_32M_2016_XTM20032000DT00351005 -> 32k; footprint Crystal:Crystal_SMD_2016-4Pin_2.0x1.6mm -> Crystal:Crystal_SMD_3215-2Pin_3.2x1.5mm
- moved Y1 116.3 mm to (115.0, 118.7), turned to 90 degrees
- moved J5 112.3 mm to (110.8, 135.5), turned to 90 degrees
- moved Y2 105.1 mm to (107.0, 129.7)
- moved R15 104.9 mm to (105.0, 119.0), turned to -90 degrees
- moved R3 104.7 mm to (104.5, 120.5), turned to 180 degrees
- moved R12 103.4 mm to (114.0, 130.5), turned to 90 degrees
- moved R16 102.6 mm to (107.3, 120.6), turned to 180 degrees
- moved L2 101.3 mm to (108.5, 118.8), turned to -90 degrees
- moved R10 100.6 mm to (109.6, 129.8), turned to 90 degrees
- moved C9 98.4 mm to (105.5, 132.1), turned to 90 degrees
- moved R9 95.4 mm to (118.7, 133.6), turned to 90 degrees
- moved C10 95.1 mm to (108.3, 132.2), turned to 90 degrees
- moved Y4 91.1 mm to (140.0, 120.2)
- moved C17 89.9 mm to (106.3, 124.9), turned to -90 degrees
- moved R4 89.5 mm to (130.7, 136.4), turned to 90 degrees
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Connections:
- net /ch584/PWM6 renamed RESET_CH5x
- net Net-(U3-GPIO9) renamed GBOOT
- C3 pad 1: Net-(J8-Pin_2) -> Net-(J16-Pin_1)
- C3 pad 2: Net-(J8-Pin_1) -> Net-(J16-Pin_2)
- C4 pad 1: Net-(J7-Pin_2) -> Net-(J15-Pin_1)
- C4 pad 2: Net-(J7-Pin_1) -> Net-(J15-Pin_2)
- C5 pad 1: Net-(J6-Pin_2) -> Net-(J14-Pin_1)
- C5 pad 2: Net-(J6-Pin_1) -> Net-(J6-Pin_2)
- C6 pad 1: unconnected-(C6-Pad1) -> Net-(J11-Pin_1)
- C6 pad 2: unconnected-(C6-Pad2) -> Net-(J11-Pin_2)
- J1 pad A6: USBDP -> /power/DPlusIn
- J1 pad A7: USBDM -> /power/DMinusIn
- J1 pad B6: USBDP -> /power/DPlusIn
- J1 pad B7: USBDM -> /power/DMinusIn
- J6 pad 1: Net-(J6-Pin_1) -> Net-(J14-Pin_1)
- J7 pad 1: Net-(J7-Pin_1) -> Net-(J15-Pin_1)
- J7 pad 2: Net-(J7-Pin_2) -> Net-(J15-Pin_2)
- J8 pad 1: Net-(J8-Pin_1) -> Net-(J16-Pin_1)
- J8 pad 2: Net-(J8-Pin_2) -> Net-(J16-Pin_2)
- R11 pad 1: Net-(U3-CHIP_EN) -> +3V3
- R11 pad 2: +3V3 -> /RESET_GLOBAL
- R4 pad 1: USBDM -> /power/DMinusIn
- R4 pad 2: Net-(U3-GPIO18) -> USBDM
- R5 pad 1: USBDP -> /power/DPlusIn
- R5 pad 2: Net-(U3-GPIO19) -> USBDP
- SW1 pad 1: Net-(U3-CHIP_EN) -> GND
- SW1 pad 2: GND -> /RESET_GLOBAL
- U2 pad 1: Net-(J6-Pin_1) -> Net-(J6-Pin_2)
- U2 pad 6: Net-(J6-Pin_2) -> Net-(J14-Pin_1)
- U3 pad 25: Net-(U3-GPIO18) -> USBDM
- U3 pad 26: Net-(U3-GPIO19) -> USBDP
- U3 pad 7: Net-(U3-CHIP_EN) -> RESET_ESP
- U4 pad 1: Net-(J7-Pin_1) -> Net-(J15-Pin_2)
- U4 pad 6: Net-(J7-Pin_2) -> Net-(J15-Pin_1)
- U5 pad 1: Net-(J8-Pin_1) -> Net-(J16-Pin_2)
- U5 pad 6: Net-(J8-Pin_2) -> Net-(J16-Pin_1)
- U6 pad 1: Net-(J11-Pin_1) -> unconnected-(U6-I/O1-Pad1)
- U6 pad 2: GND -> /power/DMinusIn
- U6 pad 3: /ch584/PWM2 -> GND
- U6 pad 4: /ch584/PWM1 -> /power/DPlusIn
- U6 pad 5: +BATT -> unconnected-(U6-I/O4-Pad5)
- U6 pad 6: Net-(J11-Pin_2) -> unconnected-(U6-NC-Pad6)
- Y1 pad 1: Net-(U8B-PA11_X32KO_TMR2) -> Net-(U3-XTAL_P)
- Y1 pad 2: Net-(U8B-PA10_X32KI_TMR1) -> GND
- Y4 pad 1: /ch584/clko -> Net-(U8B-PA11_X32KO_TMR2)
- Y4 pad 2: GND -> Net-(U8B-PA10_X32KI_TMR1)
Other:
- board outline added: 64 x 60 mm
- board text removed: "PLENTTTTTTTY OF ROOOOM"
- board text removed: "Will USB fit? or will it be pins for uart?"

Commit message: this is just getting silly
Parts:
- added H1: Mounting_SMTSO3015CTJ, jlc-extras:Mounting_SMTSO_M3, F.Cu at (160.0, 110.0)
- added H2: Mounting_SMTSO3015CTJ, jlc-extras:Mounting_SMTSO_M3, F.Cu at (104.0, 110.0)
- added JP4: KJumper_2, TestPoint:TestPoint_2Pads_Pitch2.54mm_Drill0.8mm, F.Cu at (142.5, 104.8)
- added Q1: 2N7002, Package_TO_SOT_SMD:SOT-23, F.Cu at (151.8, 108.2)
- added R13: 0R, Resistor_SMD:R_0402_1005Metric, F.Cu at (148.5, 104.0)
- added R17: 0R, Resistor_SMD:R_0402_1005Metric, F.Cu at (155.5, 104.0)
- added R18: 10k, Resistor_SMD:R_0402_1005Metric, F.Cu at (152.8, 115.0)
- moved JP3 5.26 mm to (139.8, 107.2)
- moved U9 5.01 mm to (134.5, 106.2)
- moved J7 5.00 mm to (108.9, 96.9)
- moved J15 4.65 mm to (108.5, 100.9)
- moved R16 4.60 mm to (111.9, 120.5)
- moved U2 4.40 mm to (117.2, 106.2)
- moved J6 4.25 mm to (118.9, 96.9)
- moved U5 4.10 mm to (127.2, 106.2)
- moved U4 4.06 mm to (110.0, 106.2)
- moved C6 4.05 mm to (134.5, 103.5)
- moved R15 4.01 mm to (109.0, 119.0)
- moved C18 4.00 mm to (111.3, 119.0)
- moved L2 4.00 mm to (112.5, 119.0)
- moved AE1 4.00 mm to (104.0, 125.0)
- moved AE2 4.00 mm to (160.9, 123.8)
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Connections:
- J12 pad 5: /ScopeCreep/P1_OUT -> /ScopeCreep/P1_OUT_RAW
- U3 pad 13: unconnected-(U3-MTDO-Pad13) -> /ch584/PWM3
Other:
- board size 64 x 60 mm -> 64 x 58 mm
- copper layers 2 -> 4

Commit message: "schematic complete" (lol)
but yeah, i think this is most of it?  time to maybe route shit?
Parts:
- added Q3: HL2301A, Package_TO_SOT_SMD:SOT-23, F.Cu at (150.2, 108.2)
- added Q4: HL3400A, Package_TO_SOT_SMD:SOT-23, F.Cu at (154.0, 105.4)
- added R21: 0R, Resistor_SMD:R_0402_1005Metric, F.Cu at (149.8, 104.9)
- added R22: 10k, Resistor_SMD:R_0402_1005Metric, F.Cu at (152.4, 110.5)
- Q1: value 2N7002 -> HL3400A
- moved J1 40.7 mm to (103.7, 120.6), turned to -90 degrees
- moved J4 38.5 mm to (104.4, 108.2), turned to -90 degrees
- moved R2 36.0 mm to (111.2, 123.1), turned to 0 degrees
- moved H2 34.9 mm to (136.9, 121.6)
- moved J2 32.9 mm to (109.0, 108.4), turned to 0 degrees
- moved C1 32.5 mm to (127.7, 114.7)
- moved C15 32.5 mm to (127.7, 116.7)
- moved C16 32.5 mm to (127.7, 122.7)
- moved L1 32.5 mm to (123.9, 118.7)
- moved R6 32.5 mm to (130.2, 122.5)
- moved R7 32.5 mm to (130.2, 120.5)
- moved R8 32.5 mm to (130.2, 118.5)
- moved U1 32.5 mm to (127.7, 119.7)
- moved D1 31.9 mm to (113.3, 115.7), turned to 180 degrees
- moved U6 30.0 mm to (111.4, 120.8), turned to 0 degrees
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Connections:
- H1 pad 1: (no net) -> unconnected-(H1-Pad1)
- H2 pad 1: (no net) -> unconnected-(H2-Pad1)
- Q1 pad 1: Net-(Q1-G) -> /ch584/PWM5
- Q1 pad 3: /ch584/PWM3 -> Net-(Q1-D)
- R17 pad 2: Net-(Q1-G) -> Net-(Q4-G)
- U3 pad 12: unconnected-(U3-MTCK-Pad12) -> /ch584/PWM5

Commit message: update following ERC and symbol fixes
Connections:
- net USBDM renamed USBDN
- U8 pad 20: BOOT -> GBOOT
Routing:
- net USBDP: track 0.00 -> 12.3 mm
- net USBDN: track 0.00 -> 11.8 mm
