File: hw/ktwinkler-multi-r2025-12/ktwinkler-multi-r2025-12.kicad_sch (KiCad schematic)
At the start: 11 parts, among them SW1 RESET, SW2 BOOT, SW5 MODE

Commit message: hw: save before kicad 10 upgrade
Parts:
- JP1, JP2: now left out of the parts list
Changed lines of the file:
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@@
 		(unit 1)
 		(exclude_from_sim no)
-		(in_bom yes)
+		(in_bom no)
 		(on_board yes)
 		(dnp no)
@@
 		(unit 1)
 		(exclude_from_sim no)
-		(in_bom yes)
-		(on_board yes)
-		(dnp no)
+		(in_bom no)
+		(on_board yes)
+		(dnp no)

Commit message: hw: update to kicad 10 and order
We added a late qwiic connector to the ch584 side, why not, try that out
too.  We also fixed our smtso footprint, we hope...

Fuck poking the rf more, we're yolo-poling...
Parts:
- H1, H2, H3: footprint jlc-extras:Mounting_SMTSO_M3_ALT -> jlc-extras:Mounting_SMTSO_M3_ALT2
