File: hw/ktwinkler-multi-r2025-12/leds.kicad_sch (KiCad schematic)
At the start: 12 parts, among them J11 Conn_01x02, J6 Conn_01x02, J7 Conn_01x02, J8 Conn_01x02, U2 FM116C, U4 T1016H, U5 AD116, U6 FM116C

Commit message: ktwinkler hw dev: progress stash
Changed lines of the file:
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@@
 	(text "fm116c: 0.04, 60k stock (600/800mA)\nad116: 0.04, 3k stock (1.1/2A)\nlk116: 0.04 200 stock (1A/2A)\nt1016h: 0.05 4k stock  (2.3A)\nbdr6120: 0.05 ~zero stock\ngr6205: 0.03 2k stock (200mA)\nhl116: 0.03 3k stock (500/800mA)"
 		(exclude_from_sim no)
-		(at 117.856 34.798 0)
+		(at 117.602 37.338 0)
 		(effects
 			(font
@@
 				(path "/48773b41-b773-40e2-8ba4-2e78c7a3e45f/c43f945b-11fd-4720-850e-2a9100759260"
 					(reference "C5")
+					(unit 1)
+				)
+			)
+			(project "leds"
+				(path "/9ebaab77-0759-43ea-87f9-fd126be3ebdf"
+					(reference "C?")
 					(unit 1)
 				)
@@
 				)
 			)
+			(project "leds"
+				(path "/9ebaab77-0759-43ea-87f9-fd126be3ebdf"
+					(reference "J?")
+					(unit 1)
+				)
+			)
 		)
 	)
@@
 				)
 			)
+			(project "leds"
+				(path "/9ebaab77-0759-43ea-87f9-fd126be3ebdf"
+					(reference "C?")
+					(unit 1)
+				)
+			)
 		)
 	)
@@
 				)
 			)
+			(project "leds"
+				(path "/9ebaab77-0759-43ea-87f9-fd126be3ebdf"
+					(reference "U?")
+					(unit 1)
+				)
+			)
 		)
 	)
@@
 				)
 			)
+			(project "leds"
+				(path "/9ebaab77-0759-43ea-87f9-fd126be3ebdf"
+					(reference "C?")
+					(unit 1)
+				)
+			)
 		)
 	)
@@
 				)
 			)
+			(project "leds"
+				(path "/9ebaab77-0759-43ea-87f9-fd126be3ebdf"
+					(reference "C?")
+					(unit 1)
+				)
+			)
 		)
 	)
@@
 				)
 			)
+			(project "leds"
+				(path "/9ebaab77-0759-43ea-87f9-fd126be3ebdf"
+					(reference "U?")
+					(unit 1)
+				)
+			)
 		)
 	)
@@
 				)
 			)
+			(project "leds"
+				(path "/9ebaab77-0759-43ea-87f9-fd126be3ebdf"
+					(reference "#PWR?")
+					(unit 1)
+				)
+			)
 		)
 	)
@@
 				)
 			)
+			(project "leds"
+				(path "/9ebaab77-0759-43ea-87f9-fd126be3ebdf"
+					(reference "#PWR?")
+					(unit 1)
+				)
+			)
 		)
 	)
@@
 				)
 			)
+			(project "leds"
+				(path "/9ebaab77-0759-43ea-87f9-fd126be3ebdf"
+					(reference "U?")
+					(unit 1)
+				)
+			)
 		)
 	)
@@
 				)
 			)
+			(project "leds"
+				(path "/9ebaab77-0759-43ea-87f9-fd126be3ebdf"
+					(reference "#PWR?")
+					(unit 1)
+				)
+			)
 		)
 	)
@@
 				(path "/48773b41-b773-40e2-8ba4-2e78c7a3e45f/c43f945b-11fd-4720-850e-2a9100759260"
 					(reference "#PWR04")
+					(unit 1)
+				)
+			)
+			(project "leds"
+				(path "/9ebaab77-0759-43ea-87f9-fd126be3ebdf"
+					(reference "#PWR?")
 					(unit 1)
 				)
@@
 				)
 			)
+			(project "leds"
+				(path "/9ebaab77-0759-43ea-87f9-fd126be3ebdf"
+					(reference "J?")
+					(unit 1)
+				)
+			)
 		)
 	)
@@
 				)
 			)
+			(project "leds"
+				(path "/9ebaab77-0759-43ea-87f9-fd126be3ebdf"
+					(reference "J?")
+					(unit 1)
+				)
+			)
 		)
 	)
@@
 				(path "/48773b41-b773-40e2-8ba4-2e78c7a3e45f/c43f945b-11fd-4720-850e-2a9100759260"
 					(reference "U6")
+					(unit 1)
+				)
+			)
+			(project "leds"
+				(path "/9ebaab77-0759-43ea-87f9-fd126be3ebdf"
+					(reference "U?")
 					(unit 1)
 				)
@@
 				)
 			)
-		)
-	)
+			(project "leds"
+				(path "/9ebaab77-0759-43ea-87f9-fd126be3ebdf"
+					(reference "J?")
+					(unit 1)
+				)
+			)
+		)
+	)
+	(sheet_instances
+		(path "/"
+			(page "1")
+		)
+	)
+	(embedded_fonts no)
 )

Commit message: pushing onwards like a madlad
Parts:
- removed C5, C6, C7, C8: 100nF, Capacitor_SMD:C_0603_1608Metric, symbol karl-atomic-basic:KC0603_100nF
- added C3, C4, C5, C6: 100nF, Capacitor_SMD:C_0402_1005Metric, symbol karl-atomic-basic:KC0402_100nF_16V
Connections:
- net at J7.1 (Pin_1), U4.1 (OUTB): now also C4.2
- net at J7.2 (Pin_2), U4.6 (OUTA): now also C4.1
- net at J8.2 (Pin_2), U5.6 (OUTA): now also C3.1
- net at J8.1 (Pin_1), U5.1 (OUTB): now also C3.2
- net at J6.2 (Pin_2), U2.6 (OUTA): now also C5.1
- net at J6.1 (Pin_1), U2.1 (OUTB): now also C5.2
Other:
- note added: "Try and split these power? to eval the drivers separately?"

Commit message: ready for scope creep
I think the schematic is ... mostly ok?  I need to decide how much of
the han p1 port scope creep to bother doing, or not...

I've roughyl blocked out the board, seems as good as any?
Parts:
- removed U6: FM116C, Package_TO_SOT_SMD:SOT-23-6, symbol karl-parts:FM116C
- added J13, J14, J15, J16: Conn_01x02, TestPoint:TestPoint_2Pads_Pitch2.54mm_Drill0.8mm, symbol Connector_Generic:Conn_01x02
- added JP3: LocalPower, TestPoint:TestPoint_2Pads_Pitch2.54mm_Drill0.8mm, symbol Jumper:Jumper_2_Small_Open
- added U9: GM8023B, Package_TO_SOT_SMD:SOT-23-6, symbol karl-parts:Driver_GM8023B
- J11: footprint Connector_Phoenix_MC:PhoenixContact_MCV_1,5_2-G-3.81_1x02_P3.81mm_Vertical -> Connector_Phoenix_MC:PhoenixContact_MC_1,5_2-G-3.5_1x02_P3.50mm_Horizontal; LCSC Part # C8396 -> C8387; MPN WJ15EDGVC-3.81-2P -> WJ15EDGRC-3.81-2P
- J6, J7, J8: footprint Connector_Phoenix_MC:PhoenixContact_MCV_1,5_2-G-3.81_1x02_P3.81mm_Vertical -> Connector_Phoenix_MC:PhoenixContact_MC_1,5_2-G-3.5_1x02_P3.50mm_Horizontal; LCSC Part # C8396 -> C8387
Connections:
- net GND: now also U9.2 (GND)
- net LED1A: now also U9.3 (INA)
- net LED1B: now also U9.6 (INB)
- net PWR_LEDS: now also JP3.1 (A)
- net at C4.2, U4.1 (OUTB): now also J7.2 (Pin_2), J15.2 (Pin_2); no longer J7.1 (Pin_1)
- net at C4.1, U4.6 (OUTA): now also J7.1 (Pin_1), J15.1 (Pin_1); no longer J7.2 (Pin_2)
- net at C6.1: now also J11.1 (Pin_1), J13.1 (Pin_1), U9.4 (OUTA)
- net at C6.2: now also J11.2 (Pin_2), J13.2 (Pin_2), U9.1 (OUTB)
- net at C5.1, U2.6 (OUTA): now also J6.1 (Pin_1), J14.1 (Pin_1); no longer J6.2 (Pin_2)
- net at C5.2, U2.1 (OUTB): now also J6.2 (Pin_2); no longer J6.1 (Pin_1)
- net at C3.2, U5.1 (OUTB): now also J8.2 (Pin_2), J16.2 (Pin_2); no longer J8.1 (Pin_1)
- net at C3.1, U5.6 (OUTA): now also J8.1 (Pin_1), J16.1 (Pin_1); no longer J8.2 (Pin_2)
- new net: JP3.2 (B), U9.5 (VDD)
Other:
- note added: "Allow providing other power on the jumper, this channel can do 40V, in theory..."
- note added: "put a 1x4 on each one? for extension via pins, not just the connectors?"

Commit message: update following ERC and symbol fixes
Parts:
- U2: symbol karl-parts:FM116C -> karl-parts:Driver_FM116C
- U4: symbol karl-parts:T1016H -> karl-parts:Driver_T1016H
- U5: symbol karl-parts:AD116 -> karl-parts:Driver_AD116
Connections:
- net at C5.2, J6.2 (Pin_2), U2.1 (OUTB): now also J14.2 (Pin_2)

Commit message: hw: update to kicad 10 and order
We added a late qwiic connector to the ch584 side, why not, try that out
too.  We also fixed our smtso footprint, we hope...

Fuck poking the rf more, we're yolo-poling...
Parts:
- J13, J14, J15, J16, JP3: now left out of the parts list
