File: hw/ktwinkler-multi-r2025-12/esp32.kicad_sch (KiCad schematic)
At the start: 26 parts, among them J5 Conn_01x03, J9 BWU.FL-IPEX1, U3 ESP32-C3FH4, Y1 40M, Y2 32k

Commit message: hw/multi-rev2025: flag more total fuckups in the design
lol, using 6 PWMs on the internal spi channel.  I've read that section
multiple times, and just... wot?  oh well.  Cut a few traces, can still
do some things...
Other:
- note added: "LOL, you fucking eeedjit"
Changed lines of the file:
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@@
 	(generator_version "10.0")
 	(paper "A4")
+	(text "LOL, you fucking eeedjit"
+		(exclude_from_sim no)
+		(at 178.308 122.936 0)
+		(effects
+			(font
+				(size 1.27 1.27)
+			)
+		)
+	)
 	(text "hang on....\nI was going to yolo this,\nbut.. do I need to?\nwell, what was the point otherwise?"
 		(exclude_from_sim no)
