File: hw/ktwinkler-24-basic1/leds.kicad_sch (KiCad schematic)
At the start: 17 parts, among them J11 Conn_01x02, J13 Conn_01x02, J14 Conn_01x02, J15 Conn_01x02, J16 Conn_01x02, J6 Conn_01x02, J7 Conn_01x02, J8 Conn_01x02, U2 FM116C, U4 T1016H, U5 AD116, U9 GM8023B

Commit message: ktwinkler-24: schematic "complete"
Parts:
- removed C3, C4: 100nF, Capacitor_SMD:C_0402_1005Metric, symbol karl-atomic-basic:KC0402_100nF_16V
- removed J7, J8: Conn_01x02, Connector_Phoenix_MC:PhoenixContact_MC_1,5_2-G-3.5_1x02_P3.50mm_Horizontal, symbol Connector_Generic:Conn_01x02
- removed JP3: LocalPower, TestPoint:TestPoint_2Pads_Pitch2.54mm_Drill0.8mm, symbol Jumper:Jumper_2_Small_Open
- removed U2: FM116C, Package_TO_SOT_SMD:SOT-23-6, symbol karl-parts:Driver_FM116C
- removed U4: T1016H, Package_TO_SOT_SMD:SOT-23-6, symbol karl-parts:Driver_T1016H
- removed U5: AD116, Package_TO_SOT_SMD:SOT-23-6, symbol karl-parts:Driver_AD116
- added C10, C9: 100nF, Capacitor_SMD:C_0402_1005Metric, symbol karl-atomic-basic:KC0402_100nF_16V
- added J17: Conn_01x02, TestPoint:TestPoint_2Pads_Pitch2.54mm_Drill0.8mm, symbol Connector_Generic:Conn_01x02
- added J18: Conn_01x02, Connector_Phoenix_MC:PhoenixContact_MCV_1,5_2-G-3.81_1x02_P3.81mm_Vertical, symbol Connector_Generic:Conn_01x02
- added U12, U13, U14: GM8023B, Package_TO_SOT_SMD:SOT-23-6, symbol karl-parts:Driver_GM8023B
- J11: footprint Connector_Phoenix_MC:PhoenixContact_MC_1,5_2-G-3.5_1x02_P3.50mm_Horizontal -> Connector_Phoenix_MC:PhoenixContact_MCV_1,5_2-G-3.81_1x02_P3.81mm_Vertical; LCSC Part # C8387 -> C8396; MPN WJ15EDGRC-3.81-2P -> WJ15EDGVC-3.81-02P-14-00A
- J16: footprint TestPoint:TestPoint_2Pads_Pitch2.54mm_Drill0.8mm -> Connector_Phoenix_MC:PhoenixContact_MCV_1,5_2-G-3.81_1x02_P3.81mm_Vertical; LCSC Part # (none) -> C8396; MPN (none) -> WJ15EDGVC-3.81-02P-14-00A; now in the parts list
- J6: footprint Connector_Phoenix_MC:PhoenixContact_MC_1,5_2-G-3.5_1x02_P3.50mm_Horizontal -> Connector_Phoenix_MC:PhoenixContact_MCV_1,5_2-G-3.81_1x02_P3.81mm_Vertical; LCSC Part # C8387 -> C8396; MPN WJ15EDGVC-3.81-2P -> WJ15EDGVC-3.81-02P-14-00A
Connections:
- net GND: now also U12.2 (GND), U13.2 (GND), U14.2 (GND)
- net LED2A: now also U12.3 (INA)
- net LED2B: now also U12.6 (INB)
- net LED3A: now also U13.3 (INA)
- net LED3B: now also U13.6 (INB)
- net LED4A: now also U14.3 (INA)
- net LED4B: now also U14.6 (INB)
- net PWR_LEDS: now also U9.5 (VDD), U12.5 (VDD), U13.5 (VDD), U14.5 (VDD)
- net at J15.1 (Pin_1): now also J16.1 (Pin_1), C9.1, U13.4 (OUTA)
- net at J15.2 (Pin_2): now also J16.2 (Pin_2), C9.2, U13.1 (OUTB)
- net at C5.1, J14.1 (Pin_1), J6.1 (Pin_1): now also U12.4 (OUTA)
- net at C5.2, J14.2 (Pin_2), J6.2 (Pin_2): now also U12.1 (OUTB)
- new net: C10.2, J17.2 (Pin_2), J18.2 (Pin_2), U14.1 (OUTB)
- new net: C10.1, J17.1 (Pin_1), J18.1 (Pin_1), U14.4 (OUTA)
Other:
- note removed: "Allow providing other power on the jumper, this channel can do 40V, in theory..."
- note removed: "FIXME"
- note removed: "Make all connectors here be vertical, not my normal horizontal. It's easier for the boxes to plug things that way."
- note removed: "Try and split these power? to eval the drivers separately?"

Commit message: k24-basic1: first cut layout complete
re(un)twisted all the outputs to be straight.
seems like this is all it needs... yolo?
Connections:
- net LED2A: now also U13.3 (INA); no longer U12.3 (INA)
- net LED2B: now also U13.6 (INB); no longer U12.6 (INB)
- net LED3A: now also U14.3 (INA); no longer U13.3 (INA)
- net LED3B: now also U14.6 (INB); no longer U13.6 (INB)
- net LED4A: now also U12.3 (INA); no longer U14.3 (INA)
- net LED4B: now also U12.6 (INB); no longer U14.6 (INB)
- net out3b: now reaches C10.2, J17.2 (Pin_2), J18.2 (Pin_2), U14.1 (OUTB)
- net out3a: now reaches C10.1, J17.1 (Pin_1), J18.1 (Pin_1), U14.4 (OUTA)
- net out2a: now reaches C9.1, J15.1 (Pin_1), J16.1 (Pin_1), U13.4 (OUTA)
- net out2b: now reaches C9.2, J15.2 (Pin_2), J16.2 (Pin_2), U13.1 (OUTB)
- net out1a: now reaches C6.1, J11.1 (Pin_1), J13.1 (Pin_1), U9.4 (OUTA)
- net out1b: now reaches C6.2, J11.2 (Pin_2), J13.2 (Pin_2), U9.1 (OUTB)
- net out4a: now reaches C5.1, J14.1 (Pin_1), J6.1 (Pin_1), U12.4 (OUTA)
- net out4b: now reaches C5.2, J14.2 (Pin_2), J6.2 (Pin_2), U12.1 (OUTB)
Other:
- moved on the sheet: C10, C5, C9, J14, J15, J16, J17, J18, J6, U12, U13, U14
