File: hw/ktwinkler-24-basic1/esp32.kicad_sch (KiCad schematic)
At the start: 26 parts, among them J5 Conn_01x03, J9 BWU.FL-IPEX1, U3 ESP32-C3FH4, Y1 40M, Y2 32k

Commit message: ktwinkler-24: schematic "complete"
Parts:
- removed C10, C9: 22pF, Capacitor_SMD:C_0402_1005Metric, symbol karl-atomic-basic:KC0402_22pF
- removed C18: 2.2pF, Capacitor_SMD:C_0402_1005Metric, symbol karl-atomic-basic:KC0402_2.2pF
- removed R16: 0R, Resistor_SMD:R_0402_1005Metric, symbol karl-atomic-basic:KR0402_0R
- removed TP2: TestPoint, TestPoint:TestPoint_THTPad_D1.0mm_Drill0.5mm, symbol Connector:TestPoint
- removed Y2: 32k, Crystal:Crystal_SMD_3215-2Pin_3.2x1.5mm, symbol karl-atomic-basic:Crystal_32k_3215_Q13FC13500004
- added C1, C3: 1.5pf, Capacitor_SMD:C_0402_1005Metric, symbol karl-atomic-basic:KC0402_1.5pF
- added C19: 1uF, Capacitor_SMD:C_0603_1608Metric, symbol karl-atomic-basic:KC0603_1uF
- added R19: 10k, Resistor_SMD:R_0402_1005Metric, symbol karl-atomic-basic:KR0402_10k
- L2: value 1nH -> 2.2nH; LCSC Part # C18222 -> C86061; MPN LQG15HS1N0S02D -> LQG15HS2N2S02D
- R15: now fitted
- R3: now not fitted
Connections:
- net P1IN is gone; now on net PWM8: U3.13 (MTDO)
- net P1_Req_Out is gone; now on net PWM7: U3.12 (MTCK)
- net +3V3: now also R19.2
- net GND: now also C1.2, C19.2, C3.2; no longer L2.1
- net PWM1: now also U3.9 (MTMS); no longer U3.16 (GPIO10)
- net PWM3: now also U3.4 (XTAL_32K_P); no longer U3.21 (SPICS0)
- net PWM4: now also U3.5 (XTAL_32K_N); no longer U3.22 (SPICLK)
- net PWM5: now also R12.2, U3.14 (GPIO8); no longer U3.23 (SPID)
- net PWM6: now also R10.2, U3.6 (GPIO2); no longer U3.24 (SPIQ)
- net PWM7: no longer U3.19 (SPIHD)
- net PWM8: no longer U3.20 (SPIWP)
- net at TP3.1, U3.1 (LNA_IN): now also L2.1, C3.1; no longer L2.2
- net at R15.2, R3.1: now also L2.2, C1.1
- net RESET_ESP: no longer names the net of U3.7 (CHIP_EN)
- net RESET_ESP: now also C19.1, R19.1
- no-connect marks 0 -> 6
Other:
- note added: "Internal flash don't touch!"
- note added: "Just stock c3 hw guidelines"
- note removed: "LOL, you fucking eeedjit"
- moved on the sheet: L2, R10, R12

Commit message: k24-basic1: first cut layout complete
re(un)twisted all the outputs to be straight.
seems like this is all it needs... yolo?
Parts:
- AE1: footprint RF_Experiments:ANT-YOLOPOLE -> RF_Antenna:Texas_SWRA117D_2.4GHz_Left
Connections:
- net PWM1: now also U3.5 (XTAL_32K_N); no longer U3.9 (MTMS)
- net PWM2: now also R10.2, U3.6 (GPIO2); no longer U3.10 (MTDI)
- net PWM3: now also U3.13 (MTDO); no longer U3.4 (XTAL_32K_P)
- net PWM4: now also R12.2, U3.14 (GPIO8); no longer U3.5 (XTAL_32K_N)
- net PWM5: now also U3.4 (XTAL_32K_P); no longer R12.2, U3.14 (GPIO8)
- net PWM6: now also U3.9 (MTMS); no longer R10.2, U3.6 (GPIO2)
- net PWM7: now also U3.10 (MTDI); no longer U3.12 (MTCK)
- net PWM8: now also U3.12 (MTCK); no longer U3.13 (MTDO)
- net U0RXD: now reaches J5.2 (Pin_2), U3.27 (U0RXD)
- net U0TXDb: now reaches R9.2, U3.28 (U0TXD)
- net U0TXD: now reaches J5.3 (Pin_3), R9.1
Changed lines of the file:
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@@
 	)
 	(label "PWM1"
+		(at 104.14 124.46 180)
+		(effects
+			(font
+				(size 1.27 1.27)
+			)
+			(justify right bottom)
+		)
+	)
+	(label "U0TXDb"
+		(at 102.87 114.3 0)
+		(effects
+			(font
+				(size 1.27 1.27)
+			)
+			(justify left bottom)
+		)
+	)
+	(label "PWM6"
 		(at 162.56 104.14 0)
 		(effects
@@
 		)
 	)
-	(label "PWM6"
-		(at 106.68 93.98 180)
+	(label "PWM4"
+		(at 106.68 99.06 180)
 		(effects
 			(font
@@
 		)
 	)
-	(label "PWM4"
-		(at 104.14 124.46 180)
-		(effects
-			(font
-				(size 1.27 1.27)
-			)
-			(justify right bottom)
+	(label "U0TXD"
+		(at 76.2 114.3 0)
+		(effects
+			(font
+				(size 1.27 1.27)
+			)
+			(justify left bottom)
 		)
 	)
@@
 		)
 	)
+	(label "U0RXD"
+		(at 80.01 116.84 0)
+		(effects
+			(font
+				(size 1.27 1.27)
+			)
+			(justify left bottom)
+		)
+	)
 	(label "PWM4"
 		(at 30.48 77.47 0)
@@
 	)
 	(label "PWM8"
-		(at 162.56 111.76 0)
+		(at 162.56 109.22 0)
 		(effects
 			(font
@@
 	)
 	(label "PWM7"
-		(at 162.56 109.22 0)
+		(at 162.56 106.68 0)
 		(effects
 			(font
@@
 	)
 	(label "PWM5"
-		(at 106.68 99.06 180)
+		(at 104.14 121.92 180)
 		(effects
 			(font
@@
 	)
 	(label "PWM2"
-		(at 162.56 106.68 0)
-		(effects
-			(font
-				(size 1.27 1.27)
-			)
-			(justify left bottom)
+		(at 106.68 93.98 180)
+		(effects
+			(font
+				(size 1.27 1.27)
+			)
+			(justify right bottom)
 		)
 	)
@@
 	)
 	(label "PWM3"
-		(at 104.14 121.92 180)
-		(effects
-			(font
-				(size 1.27 1.27)
-			)
-			(justify right bottom)
+		(at 162.56 111.76 0)
+		(effects
+			(font
+				(size 1.27 1.27)
+			)
+			(justify left bottom)
 		)
 	)
@@
 			)
 		)
-		(property "Footprint" "RF_Experiments:ANT-YOLOPOLE"
+		(property "Footprint" "RF_Antenna:Texas_SWRA117D_2.4GHz_Left"
 			(at 261.62 83.82 0)
 			(hide yes)

Commit message: k24-1: mounting, rounding labels
save point before retrying thigns
Parts:
- added TP4: TestPoint, TestPoint:TestPoint_Pad_D1.0mm, symbol Connector:TestPoint
Connections:
- net at U3.16 (GPIO10): now also TP4.1
Changed lines of the file:
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@@
+	(wire
+		(pts
+			(xy 92.71 104.14) (xy 109.22 104.14)
+		)
+		(stroke
+			(width 0)
+			(type default)
+		)
+	)
 	(wire
 		(pts
@@
 					(unit 1)
 				)
+			)
+		)
+	)
+	(symbol
+		(lib_id "Connector:TestPoint")
+		(at 92.71 104.14 90)
+		(unit 1)
+		(body_style 1)
+		(exclude_from_sim no)
+		(in_bom no)
+		(on_board yes)
+		(in_pos_files yes)
+		(dnp no)
+		(fields_autoplaced yes)
+		(property "Reference" "TP4"
+			(at 89.408 99.06 90)
+			(show_name no)
+			(do_not_autoplace no)
+			(effects
+				(font
+					(size 1.27 1.27)
+				)
+			)
+		)
+		(property "Value" "TestPoint"
+			(at 89.408 101.6 90)
+			(show_name no)
+			(do_not_autoplace no)
+			(effects
+				(font
+					(size 1.27 1.27)
+				)
+			)
+		)
+		(property "Footprint" "TestPoint:TestPoint_Pad_D1.0mm"
+			(at 92.71 99.06 0)
+			(hide yes)
+			(show_name no)
+			(do_not_autoplace no)
+			(effects
+				(font
+					(size 1.27 1.27)
+				)
+			)
+		)
+		(property "Datasheet" ""
+			(at 92.71 99.06 0)
+			(hide yes)
+			(show_name no)
+			(do_not_autoplace no)
+			(effects
+				(font
+					(size 1.27 1.27)
+				)
+			)
+		)
+		(property "Description" "test point"
+			(at 92.71 104.14 0)
+			(hide yes)
+			(show_name no)
+			(do_not_autoplace no)
+			(effects
+				(font
+					(size 1.27 1.27)
+				)
+			)
+		)
+		(property "Manufacturer" ""
+			(at 92.71 104.14 0)
+			(hide yes)
+			(show_name no)
+			(do_not_autoplace no)
+			(effects
+				(font
+					(size 1.27 1.27)
+				)
+			)
+		)
+		(pin "1"
+		)
+		(instances
+			(project "ktwinkler-24-basic1"
+				(path "/48773b41-b773-40e2-8ba4-2e78c7a3e45f/f1fab45e-2489-4bf6-8b0f-5e1748a9ff79"
+					(reference "TP4")
+					(unit 1)
+				)
