File: hw/ktwinkler-24-basic1/power.kicad_sch (KiCad schematic)
At the start: 24 parts, among them J1 USB_C_Receptacle_USB2.0_16P, J2 Conn_01x02, J4 Conn_01x02, U1 TPS631000DRLR, U6 Protection_H5VU25UC, U7 AMS1117-3.3, U8 SY8303

Commit message: ktwinkler-24: schematic "complete"
Parts:
- removed C1, C15, C16, C19, C20, C21: 22uF, Capacitor_SMD:C_0805_2012Metric, symbol karl-atomic-basic:KC0805_22uF_25V
- removed L1: 1uH, Inductor_SMD:L_1206_3216Metric, symbol Device:L_Small
- removed R13, R8: 220k, Resistor_SMD:R_0402_1005Metric, symbol karl-atomic-basic:KR0402_220k
- removed R17, R7: 39k, Resistor_SMD:R_0402_1005Metric, symbol karl-atomic-basic:KR0402_39k
- removed R6: 10k, Resistor_SMD:R_0402_1005Metric, symbol karl-atomic-basic:KR0402_10k
- removed U1: TPS631000DRLR, Package_TO_SOT_SMD:SOT-583-8, symbol karl-parts:TPS631000DRLR
- removed U7: AMS1117-3.3, Package_TO_SOT_SMD:SOT-223-3_TabPin2, symbol Regulator_Linear:AMS1117-3.3
- removed U8: SY8303, Package_TO_SOT_SMD:TSOT-23-8, symbol karl-parts:Buck_Regulator_SY8303_40V_3A_SOT23
- added C24, C28: 10nF, Capacitor_SMD:C_0402_1005Metric, symbol karl-atomic-basic:KC0402_10nF_50V
- added C25, C26, C31, C32: 22uF, Capacitor_SMD:C_0805_2012Metric, symbol karl-atomic-basic:KC0805_22uF_25V
- added C29, C30: 10uF, Capacitor_SMD:C_1206_3216Metric, symbol karl-atomic-basic:KC1206_10uF_50V
- added JP2, JP4, JP5, JP6, JP7: KJumper_2, Connector_PinHeader_2.54mm:PinHeader_1x02_P2.54mm_Vertical, symbol karl-parts:KJumper_2
- added L3, L4: 2u2, et-parts:L_Changjiang_FNR4030S, symbol Device:L
- added R17, R18: 7k5, Resistor_SMD:R_0402_1005Metric, symbol karl-atomic-basic:KR0402_7k5
- added R21, R24: 470R, Resistor_SMD:R_0402_1005Metric, symbol karl-atomic-basic:KR0402_470R
- added R22, R25: 220k, Resistor_SMD:R_0402_1005Metric, symbol karl-atomic-basic:KR0402_220k
- added R23, R26: 20k, Resistor_SMD:R_0402_1005Metric, symbol karl-atomic-basic:KR0402_20k
- added U10, U11: SY8303, Package_TO_SOT_SMD:TSOT-23-8, symbol karl-parts:Buck_Regulator_SY8303_40V_3A_SOT23
- J4: footprint Connector_Phoenix_MC:PhoenixContact_MC_1,5_2-G-3.5_1x02_P3.50mm_Horizontal -> Connector_Phoenix_MC:PhoenixContact_MCV_1,5_2-G-3.81_1x02_P3.81mm_Vertical; LCSC Part # C8387 -> C8396; MPN WJ15EDGVC-3.81-2P -> WJ15EDGVC-3.81-02P-14-00A
Connections:
- net +BATT is gone; now on net +VDC: D1.1 (K)
- net +VDC: now also C29.1, C30.1, JP6.2 (B), U10.5 (IN), U10.8 (EN), U11.5 (IN), U11.8 (EN)
- net GND: now also C25.2, C26.2, C29.2, C30.2, C31.2, C32.2, R17.2, R18.2, R21.2, R23.2, R24.2, R26.2, U10.3 (GND), U10.4 (GND), U11.3 (GND), U11.4 (GND)
- net VBUS: now also C25.1, C26.1, JP6.1 (A), L3.2, R22.1
- new net: JP5.1 (A), R26.1
- new net: C24.1, U10.7 (BS)
- new net: C24.2, L3.1, U10.6 (LX)
- new net: JP4.1 (A), R17.1
- new net: JP2.2 (B), JP4.2 (B), R22.2, U10.1 (FB)
- new net: R24.1, U11.2 (FS)
- new net: JP5.2 (B), JP7.2 (B), R25.2, U11.1 (FB)
- new net: JP2.1 (A), R23.1
- new net: JP7.1 (A), R18.1
- new net: C28.2, L4.1, U11.6 (LX)
- new net: C28.1, U11.7 (BS)
- new net: R21.1, U10.2 (FS)
- new net +3.3V: C31.1, C32.1, L4.2, R25.1
Other:
- note added: "1.49uH calc for 3.3, 2.2 ok? yolo boi"
- note added: "2 for 5v and 3 for 12v, 2.2 should be fine, yolo"
- note added: "5-24V in, with buck to 12 buck to 5 buck to 3.3 (lol, no, who needs that) passthrough as options for the led supply. separate 3.3V ~ish supply for the esp32 itself. just an ams1117-3.3 for the esp32? could I live with myself?"
- note added: "Fsw is 10^5 / Rfs (in kOhm) Lets say 2M, small(er) inductors => 470R -> 2.12M that'll do"
- note added: "eh, esp32 wants them, so be it"
- note removed: "5-24V in, with buck to 12 buck to 5 buck to 3.3 passthrough as options for the led supply. separate 3.3V ~ish supply for the esp32 itself. just an ams1117-3.3 for the esp32? could I live with myself?"
- note removed: "FIXME"
- note removed: "TI promises a single 0805 output, 47uf! not sure...."
- note removed: "This shit only works if you're doing vbus of 5v, like we, really, are on this board. If you do vbus of 12V, you're kinda fucked here..."
- note removed: "Worst case, we run out of time, we just do a 5V buck for leds and then 3.3 for esp32, get shit _done_ and out the door. it's already sept 17, who am I fucking kidding."
- note removed: "eh, esp32 wants them, ch58x has them internal, just slap em down"
- moved on the sheet: J2

Commit message: k24: rough blocked, fixed old values for bucks
Parts:
- removed JP5, JP7: KJumper_2, Connector_PinHeader_2.54mm:PinHeader_1x02_P2.54mm_Vertical, symbol karl-parts:KJumper_2
- removed R18: 7k5, Resistor_SMD:R_0402_1005Metric, symbol karl-atomic-basic:KR0402_7k5
- removed R22, R25: 220k, Resistor_SMD:R_0402_1005Metric, symbol karl-atomic-basic:KR0402_220k
- removed R26: 20k, Resistor_SMD:R_0402_1005Metric, symbol karl-atomic-basic:KR0402_20k
- added R6: 33k, Resistor_SMD:R_0402_1005Metric, symbol karl-atomic-basic:KR0402_33k
- added R7, R8: 150k, Resistor_SMD:R_0402_1005Metric, symbol karl-atomic-basic:KR0402_150k
Connections:
- net +3.3V: now also R7.1
- net GND: now also R6.2
- net VBUS: now also R8.1
- net at JP2.2 (B), JP4.2 (B), U10.1 (FB): now also R8.2
- net at U11.1 (FB): now also R6.1, R7.2
Other:
- note added: "so, you don't have a tvs for vbus this way?"

Commit message: k24-basic1: first cut layout complete
re(un)twisted all the outputs to be straight.
seems like this is all it needs... yolo?
Parts:
- J2: now not fitted
- U6: footprint Package_DFN_QFN:Diodes_UDFN-10_1.0x2.5mm_P0.5mm -> Package_DFN_QFN:Diodes_UDFN-10_1x2.5mm_P0.5mm
Connections:
- net VBUS: no longer D1.2 (A), J1.A4 (VBUS), J1.A9 (VBUS), J1.B4 (VBUS), J1.B9 (VBUS)
- net +3.3V renamed +3V3
- new net VUBus: D1.2 (A), J1.A4 (VBUS), J1.A9 (VBUS), J1.B4 (VBUS), J1.B9 (VBUS)
Changed lines of the file:
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@@
 	(text "LMR33630BDDAR? 24V solid, 3A, 1.2Mhz, cheap and well stocked...\nLMR41420Y - 24V, 2A, 1.1Mhz, cheap and well stocked.\nSY8303 - 24v solid, 3A, 500-2000k, cheap and well stocked.\nI still refuse to use non-synch buck in the year of our wonder, 2026\nUsing two of the same, would save me extended fees, ok for small orders?\nbut just an 1117 is better?\n\n2 of them means you can always have 3.3v regardless of bus voltage?"
 		(exclude_from_sim no)
-		(at 294.894 142.24 0)
+		(at 204.47 67.056 0)
 		(effects
 			(font
@@
 	(text "5-24V in, with\n buck to 12\n buck to 5\n buck to 3.3 (lol, no, who needs that)\n passthrough\nas options for the led supply.\nseparate 3.3V ~ish supply for the esp32 itself.\njust an ams1117-3.3 for the esp32? could I live with myself?"
 		(exclude_from_sim no)
-		(at 187.452 153.162 0)
+		(at 85.598 104.14 0)
 		(effects
 			(font
@@
 		)
 	)
-	(label "VBUS"
+	(label "VUBus"
 		(at 114.3 43.18 0)
 		(effects
@@
 		(on_board yes)
 		(in_pos_files yes)
-		(dnp no)
+		(dnp yes)
 		(fields_autoplaced yes)
 		(property "Reference" "J2"
@@
 			)
 		)
-		(property "Footprint" "Package_DFN_QFN:Diodes_UDFN-10_1.0x2.5mm_P0.5mm"
+		(property "Footprint" "Package_DFN_QFN:Diodes_UDFN-10_1x2.5mm_P0.5mm"
 			(at 124.46 68.58 0)
 			(hide yes)
@@
 	)
 	(symbol
-		(lib_id "karl-atomic-basic:Diode_SS34")
-		(at 137.16 43.18 180)
+		(lib_id "power:+3V3")
+		(at 165.1 152.4 0)
 		(unit 1)
 		(body_style 1)
@@
 		(dnp no)
 		(fields_autoplaced yes)
-		(property "Reference" "D1"
-			(at 137.4775 36.83 0)
+		(property "Reference" "#PWR041"
+			(at 165.1 156.21 0)
+			(hide yes)
 			(show_name no)
 			(do_not_autoplace no)
@@
 			)
 		)
-		(property "Value" "SS34"
-			(at 137.4775 39.37 0)
+		(property "Value" "+3V3"
+			(at 165.1 147.32 0)
 			(show_name no)
 			(do_not_autoplace no)
@@
 			)
 		)
-		(property "Footprint" "Diode_SMD:D_SMA"
-			(at 137.16 38.735 0)
+		(property "Footprint" ""
+			(at 165.1 152.4 0)
 			(hide yes)
 			(show_name no)
@@
 			)
 		)
-		(property "Datasheet" "https://jlcpcb.com/api/file/downloadByFileSystemAccessId/8586172667489079296"
-			(at 137.16 43.18 0)
+		(property "Datasheet" ""
+			(at 165.1 152.4 0)
 			(hide yes)
 			(show_name no)
@@
 			)
 		)
-		(property "Description" "40V 3A Schottky Barrier Rectifier Diode, SMA"
-			(at 137.16 43.18 0)
+		(property "Description" "Power symbol creates a global label with name \"+3V3\""
+			(at 165.1 152.4 0)
 			(hide yes)
 			(show_name no)
@@
 			)
 		)
-		(property "LCSC Part #" "C8678"
-			(at 137.16 43.18 0)
-			(hide yes)
+		(pin "1"
+		)
+		(instances
+			(project "ktwinkler-24-basic1"
+				(path "/48773b41-b773-40e2-8ba4-2e78c7a3e45f/974aa20f-6384-4103-a4af-e95b95e9bb34"
+					(reference "#PWR041")
+					(unit 1)
+				)
+			)
+		)
+	)
+	(symbol
+		(lib_id "karl-atomic-basic:Diode_SS34")
+		(at 137.16 43.18 180)
+		(unit 1)
+		(body_style 1)
+		(exclude_from_sim no)
+		(in_bom yes)
+		(on_board yes)
+		(in_pos_files yes)
+		(dnp no)
+		(fields_autoplaced yes)
+		(property "Reference" "D1"
+			(at 137.4775 36.83 0)
 			(show_name no)
 			(do_not_autoplace no)
@@
 			)
 		)
-		(property "jlcbasic" "basic"
-			(at 137.16 43.18 0)
-			(hide yes)
+		(property "Value" "SS34"
+			(at 137.4775 39.37 0)
 			(show_name no)
 			(do_not_autoplace no)
@@
 			)
 		)
-		(property "MPN" "SS34"
-			(at 137.16 43.18 0)
+		(property "Footprint" "Diode_SMD:D_SMA"
+			(at 137.16 38.735 0)
 			(hide yes)
 			(show_name no)
@@
 			)
 		)
-		(property "Manufacturer" ""
+		(property "Datasheet" "https://jlcpcb.com/api/file/downloadByFileSystemAccessId/8586172667489079296"
 			(at 137.16 43.18 0)
 			(hide yes)
@@
 			)
 		)
-		(pin "2"
-		)
-		(pin "1"
-		)
-		(instances
-			(project "ktwinkler-24-basic1"
-				(path "/48773b41-b773-40e2-8ba4-2e78c7a3e45f/974aa20f-6384-4103-a4af-e95b95e9bb34"
-					(reference "D1")
-					(unit 1)
-				)
-			)
-		)
-	)
-	(symbol
-		(lib_id "power:+3.3V")
-		(at 165.1 152.4 0)
-		(unit 1)
-		(body_style 1)
-		(exclude_from_sim no)
-		(in_bom yes)
-		(on_board yes)
-		(in_pos_files yes)
-		(dnp no)
-		(fields_autoplaced yes)
-		(property "Reference" "#PWR022"
-			(at 165.1 156.21 0)
+		(property "Description" "40V 3A Schottky Barrier Rectifier Diode, SMA"
+			(at 137.16 43.18 0)
 			(hide yes)
 			(show_name no)
@@
 			)
 		)
-		(property "Value" "+3.3V"
-			(at 165.1 147.32 0)
+		(property "LCSC Part #" "C8678"
+			(at 137.16 43.18 0)
+			(hide yes)
 			(show_name no)
 			(do_not_autoplace no)
@@
 			)
 		)
-		(property "Footprint" ""
-			(at 165.1 152.4 0)
+		(property "jlcbasic" "basic"
+			(at 137.16 43.18 0)
 			(hide yes)
 			(show_name no)
@@
 			)
 		)
-		(property "Datasheet" ""
-			(at 165.1 152.4 0)
+		(property "MPN" "SS34"
+			(at 137.16 43.18 0)
 			(hide yes)
 			(show_name no)
@@
 			)
 		)
-		(property "Description" "Power symbol creates a global label with name \"+3.3V\""
-			(at 165.1 152.4 0)
+		(property "Manufacturer" ""
+			(at 137.16 43.18 0)
 			(hide yes)
 			(show_name no)
@@
 			)
 		)
+		(pin "2"
+		)
 		(pin "1"
 		)
@@
 			(project "ktwinkler-24-basic1"
 				(path "/48773b41-b773-40e2-8ba4-2e78c7a3e45f/974aa20f-6384-4103-a4af-e95b95e9bb34"
-					(reference "#PWR022")
+					(reference "D1")
 					(unit 1)
 				)

Commit message: k24-1: mounting, rounding labels
save point before retrying thigns
Connections:
- net GND: now also J1.SH (SHIELD); no longer J1.S1 (SHIELD)
Changed lines of the file:
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@@
 		(pin "B6"
 		)
-		(pin "S1"
+		(pin "SH"
 		)
 		(pin "B1"
